File: Tiboard/Tiboard-v2.1.kicad_sch (KiCad schematic)
At the start: 106 parts, among them J1 Conn_01x04, J2 USB_C_Receptacle_USB2.0, J4 Conn_01x02, J5 USB_C_Receptacle_USB2.0, J6 Conn_01x02, Q1 AO3407, Q2 AO3407, SW1 SW_PUSH_LED, SW10 SW_PUSH_LED, SW11 SW_PUSH_LED, SW12 SW_PUSH_LED, SW13 SW_PUSH_LED, SW14 SW_PUSH_LED, SW15 SW_PUSH_LED, SW16 SW_PUSH_LED, SW17 SW_PUSH_LED, SW18 SW_PUSH_LED, SW19 SW_PUSH_LED, SW2 SW_PUSH_LED, SW20 SW_PUSH_LED, SW21 SW_PUSH_LED, SW22 SW_PUSH_LED, SW23 SW_PUSH_LED, SW24 SW_PUSH_LED, SW25 Rotary_Encoder_Switch, SW26 SW_PUSH_LED, SW27 SW_PUSH_LED, SW28 SW_PUSH_LED, SW29 SW_PUSH_LED, SW3 SW_PUSH_LED, SW30 SW_PUSH_LED, SW31 SW_SPST, SW4 SW_PUSH_LED, SW5 SW_PUSH_LED, SW6 SW_PUSH_LED, SW7 SW_PUSH_LED, SW8 SW_PUSH_LED, SW9 SW_PUSH_LED, U1 E73-2G4M08S1C, U2 AP2112K-3.3, U3 TP4054, X1 32768kHz

Commit message: day1 for Tiboard V2
Parts:
- removed D1, D10, D11, D12, D13, D14, D15, D16, D17, D18, D19, D2, D20, D21, D22, D23, D24, D25, D26, D27, D28, D29, D3, D30, D4, D5, D6, D7, D8, D9: D, myboard:crkbd-diode-wz-via, symbol Device:D
- removed D31: 1N5819, Diode_SMD:D_SOD-323F, symbol nrfmicro-rescue:MBR0520
- removed D32: BLUE, LED_SMD:LED_0603_1608Metric, symbol Device:LED
- removed D33: RED, LED_SMD:LED_0603_1608Metric, symbol Device:LED
- removed J1: Conn_01x04, myboard:connector_swd, symbol Connector_Generic:Conn_01x04
- removed J2, J5: USB_C_Receptacle_USB2.0, Connector_USB:USB_C_Receptacle_HRO_TYPE-C-31-M-12, symbol Connector:USB_C_Receptacle_USB2.0
- removed J4, J6: Conn_01x02, Connector_JST:JST_SH_SM02B-SRSS-TB_1x02-1MP_P1.00mm_Horizontal, symbol Connector_Generic:Conn_01x02
- removed JP9: SolderJumper_2_Open, Jumper:SolderJumper-2_P1.3mm_Open_RoundedPad1.0x1.5mm, symbol Jumper:SolderJumper_2_Open
- removed Q1, Q2: AO3407, Package_TO_SOT_SMD:SOT-23, symbol nrfmicro-rescue:BSS83P
- removed R10, R11: 5.1K, Resistor_SMD:R_0603_1608Metric, symbol Device:R
- removed R12, R13: 4.7K, Resistor_SMD:R_0603_1608Metric, symbol Device:R
- removed R14: 100k, Resistor_SMD:R_0603_1608Metric, symbol Device:R
- removed R4, R7: 1K, Resistor_SMD:R_0603_1608Metric, symbol Device:R
- removed R5: 820K, Resistor_SMD:R_0603_1608Metric, symbol Device:R
- removed R6, R8: 2M, Resistor_SMD:R_0603_1608Metric, symbol Device:R
- removed R9: RPROG, Resistor_SMD:R_0603_1608Metric, symbol Device:R
- removed SW31: SW_SPST, Button_Switch_THT:SW_Slide_1P2T_CK_OS102011MS2Q, symbol Switch:SW_SPST
- removed TP4: VCC, TestPoint:TestPoint_Pad_1.0x1.0mm, symbol Connector:TestPoint
- removed TP7: DATA, TestPoint:TestPoint_Pad_1.0x1.0mm, symbol Connector:TestPoint
- removed U1: E73-2G4M08S1C, myboard:E73-2G4M08S1C-52840, symbol nrfmicro:E73-2G4M08S1C-52840
- removed U2: AP2112K-3.3, Package_TO_SOT_SMD:SOT-23-5, symbol Regulator_Linear:AP2112K-3.3
- removed U3: TP4054, Package_TO_SOT_SMD:SOT-23-5, symbol Battery_Management:MCP73832-2-OT
- removed X1: 32768kHz, Crystal:Crystal_SMD_MicroCrystal_CM9V-T1A-2Pin_1.6x1.0mm, symbol Device:Crystal_Small
- added D1, D10, D11, D12, D13, D14, D2, D3, D31, D4, D5, D6, D7, D8, D9: BAV70, Package_TO_SOT_SMD:SOT-23, symbol Diode:BAV70
- added J1: Conn_01x02_MountingPin, Connector_JST:JST_SHL_SM02B-SHLS-TF_1x02-1MP_P1.00mm_Horizontal, symbol Connector_Generic_MountingPin:Conn_01x02_MountingPin
- added J2: Conn_01x05_MountingPin, 0_Tiboard:NICEVIEW_5Pin, symbol Connector_Generic:Conn_01x05
- added R1, R2: 4.7K, Resistor_SMD:R_0603_1608Metric, symbol Device:R
- added SW31: SW_SPDT, Button_Switch_THT:SW_Slide_SPDT_Angled_CK_OS102011MA1Q, symbol Switch:SW_SPDT
- added U1: ~, 0_Tiboard:52840NANO_V2, symbol 0_Tiboard:52840NANO_V2
- H1: value MountingHole -> PointingStick; footprint myboard:Pointing_Stick -> 0_Tiboard:Pointing_Stick; now left out of the parts list
- H2, H3, H4, H5, H6, H7, H8: footprint MountingHole:MountingHole_3.2mm_M3 -> MountingHole:MountingHole_3.2mm_M3_Pad_Via; now left out of the parts list
- R3: value 100K -> 100k
- SW1, SW10, SW11, SW12, SW13, SW14, SW15, SW16, SW17, SW18, SW19, SW2, SW20, SW21, SW22, SW23, SW24, SW26, SW27, SW28, SW29, SW3, SW30, SW4, SW5, SW6, SW7, SW8, SW9: footprint myboard:Choc_Hotswap_SK6812MiniE_trace -> 0_Tiboard:TTC_mini
- TP1: value CLK -> GND
- TP2: value DATA -> CLK
- TP3: value RST -> DATA
- TP5: value GND -> VCC
- TP6: value CLK -> RST
Connections:
- net VBUS is gone; now on net GND: R3.1
- net ENCA: now also U1.5 (P0.31/AIN7)
- net ENCB: now also U1.6 (P0.29/AIN5)
- net GND: now also TP1.1, J2.4 (Pin_4), U1.15 (GND), U1.16 (GND), U1.2 (GND); no longer R3.2, TP5.1
- net LED: now also U1.19 (P0.22)
- net RESET: now also U1.3 (P0.18/RESET)
- net SW25A: now also U1.12 (P1.09/NFC1)
- net SW25B: now also D9.1 (A)
- net VCC: now also U1.4 (VCC_EXT)
- net col0: now also U1.7 (P0.02/AIN0)
- net col1: now also U1.8 (P1.15)
- net col2: now also U1.9 (P1.13)
- net col3: now also U1.10 (P1.11)
- net col4: now also U1.11 (P1.10/NFC2)
- net row0: now also D1.3 (K), D2.3 (K), D31.3 (K), U1.20 (P0.24)
- net row1: now also D3.3 (K), D4.3 (K), D5.3 (K), U1.21 (P1.00)
- net row2: now also D6.3 (K), D7.3 (K), D8.3 (K), U1.22 (P0.11)
- net row3: now also D10.3 (K), D11.3 (K), D9.3 (K), U1.23 (P1.04)
- net row4: now also D12.3 (K), D13.3 (K), D14.3 (K), U1.24 (P1.06)
- net at SW26.5: now also D12.1 (A)
- net at SW1.5: now also D31.1 (A)
- net at SW2.5: now also D31.2 (A)
- net at SW3.5: now also D1.1 (A)
- net at SW4.5: now also D1.2 (A)
- net at SW5.5: now also D2.1 (A)
- net at SW6.5: now also D2.2 (A)
- net at SW8.5: now also D3.2 (A)
- net at SW9.5: now also D4.1 (A)
- net at SW10.5: now also D4.2 (A)
- net at SW11.5: now also D5.1 (A)
- net at SW12.5: now also D5.2 (A)
- net at SW7.5: now also D3.1 (A)
- net at SW13.5: now also D6.1 (A)
- net at SW14.5: now also D6.2 (A)
- net at SW15.5: now also D7.1 (A)
- net at SW16.5: now also D7.2 (A)
- net at SW17.5: now also D8.1 (A)
- net at SW18.5: now also D8.2 (A)
- net at SW21.5: now also D10.2 (A)
- net at SW22.5: now also D11.1 (A)
- net at SW23.5: now also D14.1 (A)
- net at SW24.5: now also D11.2 (A)
- net at SW20.5: now also D10.1 (A)
- net at SW19.5: now also D9.2 (A)
- net at SW27.5: now also D12.2 (A)
- net at SW28.5: now also D13.1 (A)
- net at SW29.5: now also D13.2 (A)
- net at SW30.5: now also D14.2 (A)
- net at SW6.2 (DOUT): now also SW12.4 (DIN)
- net at SW6.4 (DIN): now also SW17.2 (DOUT); no longer SW12.2 (DOUT)
- net at SW18.2 (DOUT): now also SW24.4 (DIN); no longer SW12.4 (DIN)
- net at SW18.4 (DIN): now also SW12.2 (DOUT); no longer SW24.2 (DOUT)
- net at SW20.4 (DIN): now also SW19.2 (DOUT); no longer SW23.2 (DOUT)
- net at SW30.2 (DOUT): no longer SW23.4 (DIN)
- net at SW28.4 (DIN): now also SW24.2 (DOUT); no longer SW19.2 (DOUT)
- net at SW30.4 (DIN): now also SW23.2 (DOUT); no longer SW29.2 (DOUT)
- net at TP6.1: now also C1.2, R3.2; no longer TP1.1
- net TP_DATA_P0.08: now reaches TP3.1
- net TP_DATA_P0.08: now also R2.1, U1.14 (P0.08); no longer C1.2
- net TP_CLK_P0.20: now reaches TP2.1
- net TP_CLK_P0.20: now also R1.1
- net nRF_VDD renamed V_BAT
- net V_BAT: now also TP5.1, J2.3 (Pin_3), R1.2, R2.2, SW31.1 (A), U1.1 (B+)
- new net: J1.1 (Pin_1), SW31.2 (B)
- new net: SW23.4 (DIN), SW29.2 (DOUT)
- new net MOSI: J2.1 (Pin_1), U1.17 (P0.17)
- new net P0.06: J2.5 (Pin_5), U1.13 (P0.06)
- new net SCK: J2.2 (Pin_2), U1.18 (P0.20)
- no-connect marks 5 -> 0
Other:
- note added: "NICE!NANO"
- note removed: "1.4.x"
- note removed: "Battery monitor"
- note removed: "E73-2G4M08S1C pins: P0.02 P0.03 P0.04 P0.05 P0.06 P0.07 P0.08 P0.09 P0.10 P0.12 P0.13 P0.15 P0.17 P0.18 P0.20 P0.22 P0.24 P0.26 P0.28 P0.29 P0.30 P0.31 P1.00 P1.02 P1.04 P1.06 P1.09 P1.10 P1.11 P1.13"
- note removed: "Feather pins: P1.15 LED1 x P1.10 LED2 P0.15 BTN1 P0.19 BTN2 x P0.16 NEOPIXEL x P0.08 RX P0.06 TX P1.02 DFU P0.18 RESET"
- note removed: "Jan 3, 2021"
- note removed: "LiPo Charging"
- note removed: "Power and Filtering"
- note removed: "RProg = 1000/iBat iBat in amps RProg iBAT 10k 100mA 5k 200mA 2.5k 400mA 2k 500mA 1.25k 800mA"
- note removed: "https://github.com/joric/jorne/wiki/Trackpoint"
- note removed: "nrfmicro"
- moved on the sheet: H1, H2, H3, H4, H5, H6, H7, H8, RSW1, RSW2, SW10A, SW10B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
